Commit message: urdf_modif

File: ur5_description_custom/urdf/new_ur.urdf.xacro (robot description, xacro)
@@ -2,10 +2,9 @@
 <robot xmlns:xacro="http://wiki.ros.org/xacro" name="$(arg name)">
    <!-- robot name parameter -->
-   <xacro:arg name="name" default="ur"/>
+   <xacro:arg name="name" default="ur5_with_pen"/>
    <!-- import main macro -->
    <xacro:include filename="$(find ur_description)/urdf/ur_macro.xacro"/>
    <!-- possible 'ur_type' values: ur3, ur5, ur10, ur3e, ur5e, ur7e, ur10e, ur12e, ur16e, ur8long, ur15, ur18, ur20, ur30 -->
-   <!-- the default value should raise an error in case this was called without defining the type -->
-   <xacro:arg name="ur_type" default="ur5x"/>
+   <xacro:arg name="ur_type" default="ur5"/>
    <!-- parameters -->
    <xacro:arg name="tf_prefix" default="" />
@@ -18,13 +17,35 @@
    <xacro:arg name="safety_pos_margin" default="0.15"/>
    <xacro:arg name="safety_k_position" default="20"/>
-   <!--When using gazebo simulations absolute paths are necessary.-->
    <xacro:arg name="force_abs_paths" default="false" />
    <!-- create link fixed to the "world" -->
    <link name="world" />
+     <!-- table -->
+  <link name="table_link">
+    <visual>
+      <origin xyz="0 0 1.0" rpy="0 0 0"/>
+      <geometry>
+        <box size="0.8 0.8 1.0"/>
+      </geometry>
+      <material name="brown">
+        <color rgba="0.5 0.3 0.1 1.0"/>
+      </material>
+    </visual>
+    <collision>
+      <origin xyz="0 0 1.0" rpy="0 0 0"/>
+      <geometry>
+        <box size="0.8 0.8 1.0"/>
+      </geometry>
+    </collision>
+  </link>
+  <joint name="world_table_joint" type="fixed">
+    <parent link="world"/>
+    <child  link="table_link"/>
+    <origin xyz="0 0 0" rpy="0 0 0"/>
+  </joint>
    <!-- arm -->
    <xacro:ur_robot
      name="$(arg name)"
      tf_prefix="$(arg tf_prefix)"
-     parent="world"
+     parent="table_link"
      joint_limits_parameters_file="$(arg joint_limit_params)"
      kinematics_parameters_file="$(arg kinematics_params)"
@@ -34,7 +55,30 @@
      safety_pos_margin="$(arg safety_pos_margin)"
      safety_k_position="$(arg safety_k_position)"
-     force_abs_paths="$(arg force_abs_paths)"
-     >
-     <origin xyz="0 0 0" rpy="0 0 0" />          <!-- position robot in the world -->
+     force_abs_paths="$(arg force_abs_paths)">
+     <origin xyz="0 0 0" rpy="0 0 0" />
    </xacro:ur_robot>
+   <!-- ===== VOTRE STYLO / PINCE SIMPLIFIÉE ICI ===== -->
+   <link name="pen_link">
+     <visual>
+       <origin xyz="0 0 0.135" rpy="0 0 0"/>
+       <geometry>
+         <cylinder radius="0.1" length="0.270"/>
+       </geometry>
+       <material name="blue">
+         <color rgba="0.2 0.2 0.8 1.0"/>
+       </material>
+     </visual>
+     <collision>
+       <origin xyz="0 0 0.135" rpy="0 0 0"/>
+       <geometry>
+         <cylinder radius="0.1" length="0.27"/>
+       </geometry>
+     </collision>
+   </link>
+   <joint name="pen_fixed_joint" type="fixed">
+     <parent link="${tf_prefix}tool0"/>
+     <child  link="pen_link"/>
+     <!-- ajustez xyz/rpy pour que le stylo corresponde à la réalité -->
+     <origin xyz="0 0 0" rpy="0 0 0"/>
+   </joint>
 </robot>

Commit message: des problèmes

File: ur5_description_custom/urdf/new_ur.urdf.xacro (robot description, xacro)
@@ -1,84 +1,21 @@
 <?xml version="1.0"?>
-<robot xmlns:xacro="http://wiki.ros.org/xacro" name="ur5_avec_effecteur">
-   <!-- robot name parameter -->
-   <!--xacro:arg name="name" default="ur5_with_pen"/-->
-   <!-- import main macro -->
-   <xacro:include filename="$(find ur_description)/urdf/ur_macro.xacro"/>
-   <!-- possible 'ur_type' values: ur3, ur5, ur10, ur3e, ur5e, ur7e, ur10e, ur12e, ur16e, ur8long, ur15, ur18, ur20, ur30 -->
-   <xacro:arg name="ur_type" default="ur5"/>
-   <!-- parameters -->
-   <xacro:arg name="tf_prefix" default="" />
-   <xacro:arg name="joint_limit_params" default="$(find ur_description)/config/$(arg ur_type)/joint_limits.yaml"/>
-   <xacro:arg name="kinematics_params" default="$(find ur_description)/config/$(arg ur_type)/default_kinematics.yaml"/>
-   <xacro:arg name="physical_params" default="$(find ur_description)/config/$(arg ur_type)/physical_parameters.yaml"/>
-   <xacro:arg name="visual_params" default="$(find ur_description)/config/$(arg ur_type)/visual_parameters.yaml"/>
-   <xacro:arg name="transmission_hw_interface" default=""/>
-   <xacro:arg name="safety_limits" default="false"/>
-   <xacro:arg name="safety_pos_margin" default="0.15"/>
-   <xacro:arg name="safety_k_position" default="20"/>
-   <xacro:arg name="force_abs_paths" default="false" />
-   <!-- create link fixed to the "world" -->
-   <link name="world" />
-     <!-- table -->
-  <link name="table_link">
-    <visual>
-      <origin xyz="0 0 1.0" rpy="0 0 0"/>
-      <geometry>
-        <box size="0.8 0.8 1.0"/>
-      </geometry>
-      <material name="brown">
-        <color rgba="0.5 0.3 0.1 1.0"/>
-      </material>
-    </visual>
-    <collision>
-      <origin xyz="0 0 1.0" rpy="0 0 0"/>
-      <geometry>
-        <box size="0.8 0.8 1.0"/>
-      </geometry>
-    </collision>
-  </link>
-  <joint name="world_table_joint" type="fixed">
-    <parent link="world"/>
-    <child  link="table_link"/>
-    <origin xyz="0 0 0" rpy="0 0 0"/>
-  </joint>
-   <!-- arm -->
-   <xacro:ur_robot
-     name="ur5_avec_effecteur"
-     tf_prefix="$(arg tf_prefix)"
-     parent="table_link"
-     joint_limits_parameters_file="$(arg joint_limit_params)"
-     kinematics_parameters_file="$(arg kinematics_params)"
-     physical_parameters_file="$(arg physical_params)"
-     visual_parameters_file="$(arg visual_params)"
-     safety_limits="$(arg safety_limits)"
-     safety_pos_margin="$(arg safety_pos_margin)"
-     safety_k_position="$(arg safety_k_position)"
-     force_abs_paths="$(arg force_abs_paths)">
-     <origin xyz="0 0 0" rpy="0 0 0" />
-   </xacro:ur_robot>
-   <!-- ===== VOTRE STYLO / PINCE SIMPLIFIÉE ICI ===== -->
-   <link name="pen_link">
-     <visual>
-       <origin xyz="0 0 0.135" rpy="0 0 0"/>
-       <geometry>
-         <cylinder radius="0.1" length="0.270"/>
-       </geometry>
-       <material name="blue">
-         <color rgba="0.2 0.2 0.8 1.0"/>
-       </material>
-     </visual>
-     <collision>
-       <origin xyz="0 0 0.135" rpy="0 0 0"/>
-       <geometry>
-         <cylinder radius="0.1" length="0.27"/>
-       </geometry>
-     </collision>
-   </link>
-   <joint name="pen_fixed_joint" type="fixed">
-     <parent link="${tf_prefix}tool0"/>
-     <child  link="pen_link"/>
-     <!-- ajustez xyz/rpy pour que le stylo corresponde à la réalité -->
-     <origin xyz="0 0 0" rpy="0 0 0"/>
-   </joint>
+<robot name="robot_cell" xmlns:xacro="http://ros.org/wiki/xacro">
+  <xacro:include filename="$(find my_robot_cell_description)/urdf/my_robot_cell_macro.xacro"/>
+  <xacro:arg name="ur_type" default="ur20"/>
+  <xacro:arg name="joint_limits_parameters_file" default="$(find ur_description)/config/$(arg ur_type)/joint_limits.yaml"/>
+  <xacro:arg name="kinematics_parameters_file" default="$(find ur_description)/config/$(arg ur_type)/default_kinematics.yaml"/>
+  <xacro:arg name="physical_parameters_file" default="$(find ur_description)/config/$(arg ur_type)/physical_parameters.yaml"/>
+  <xacro:arg name="visual_parameters_file" default="$(find ur_description)/config/$(arg ur_type)/visual_parameters.yaml"/>
+  <link name="world"/>
+  <!--This will create the scene where the robot is located in-->
+  <xacro:robot_cell
+    parent="world"
+    ur_type="$(arg ur_type)"
+    joint_limits_parameters_file="$(arg joint_limits_parameters_file)"
+    kinematics_parameters_file="$(arg kinematics_parameters_file)"
+    physical_parameters_file="$(arg physical_parameters_file)"
+    visual_parameters_file="$(arg visual_parameters_file)"
+    >
+      <origin xyz="0 0 1" rpy="0 0 0" />
+  </xacro:robot_cell>
 </robot>
