Commit message: tool0

File: ur5_description_custom/urdf/robot_cell.xacro (robot description, xacro)
@@ -69,5 +69,5 @@
    </link>
    <joint name="pen_fixed_joint" type="fixed">
-     <parent link="${tf_prefix}tool0"/>
+     <parent link="$tool0"/>
      <child  link="pen_link"/>
      <!-- ajustez xyz/rpy pour que le stylo corresponde à la réalité -->

Commit message: re tool

File: ur5_description_custom/urdf/robot_cell.xacro (robot description, xacro)
@@ -69,5 +69,5 @@
    </link>
    <joint name="pen_fixed_joint" type="fixed">
-     <parent link="$tool0"/>
+     <parent link="tool0"/>
      <child  link="pen_link"/>
      <!-- ajustez xyz/rpy pour que le stylo corresponde à la réalité -->

Commit message: oskour

File: ur5_description_custom/urdf/robot_cell.xacro (robot description, xacro)
@@ -6,4 +6,5 @@
     *origin
     ur_type
+    tf_prefix
     joint_limits_parameters_file
     kinematics_parameters_file
@@ -69,5 +70,5 @@
    </link>
    <joint name="pen_fixed_joint" type="fixed">
-     <parent link="tool0"/>
+     <parent link="${tf_prefix}tool0"/>
      <child  link="pen_link"/>
      <!-- ajustez xyz/rpy pour que le stylo corresponde à la réalité -->

Commit message: sans pince

File: ur5_description_custom/urdf/robot_cell.xacro (robot description, xacro)
@@ -69,10 +69,4 @@
      </collision>
    </link>
-   <joint name="pen_fixed_joint" type="fixed">
-     <parent link="${tf_prefix}tool0"/>
-     <child  link="pen_link"/>
-     <!-- ajustez xyz/rpy pour que le stylo corresponde à la réalité -->
-     <origin xyz="0 0 0" rpy="0 0 0"/>
-   </joint>
   </xacro:macro>
 </robot>

Commit message: des

File: ur5_description_custom/urdf/robot_cell.xacro (robot description, xacro)
@@ -52,21 +52,4 @@
       <origin xyz="0 0 0" rpy="0 0 0" />
     </xacro:ur_robot>
-    <link name="pen_link">
-     <visual>
-       <origin xyz="0 0 0.135" rpy="0 0 0"/>
-       <geometry>
-         <cylinder radius="0.1" length="0.270"/>
-       </geometry>
-       <material name="blue">
-         <color rgba="0.2 0.2 0.8 1.0"/>
-       </material>
-     </visual>
-     <collision>
-       <origin xyz="0 0 0.135" rpy="0 0 0"/>
-       <geometry>
-         <cylinder radius="0.1" length="0.27"/>
-       </geometry>
-     </collision>
-   </link>
   </xacro:macro>
 </robot>

Commit message: pos

File: ur5_description_custom/urdf/robot_cell.xacro (robot description, xacro)
@@ -19,5 +19,5 @@
     <link name="table">
       <visual>
-      <origin xyz="0 0 1.0" rpy="0 0 0"/>
+      <origin xyz="0 0 0" rpy="0 0 0"/>
       <geometry>
         <box size="0.8 0.8 1.0"/>
@@ -28,5 +28,5 @@
     </visual>
     <collision>
-      <origin xyz="0 0 1.0" rpy="0 0 0"/>
+      <origin xyz="0 0 0" rpy="0 0 0"/>
       <geometry>
         <box size="0.8 0.8 1.0"/>
@@ -38,5 +38,5 @@
       <parent link="table"/>
       <child link="robot_mount"/>
-      <origin xyz="0.845 0.85 0" rpy="0 0 ${pi}" />
+      <origin xyz="0 0 1.0" rpy="0 0 0" />
     </joint>
     <!--This will create the specific robot-->

Commit message: ur5

File: ur5_description_custom/urdf/robot_cell.xacro (robot description, xacro)
@@ -52,4 +52,27 @@
       <origin xyz="0 0 0" rpy="0 0 0" />
     </xacro:ur_robot>
+    <link name="pen_link">
+     <visual>
+       <origin xyz="0 0 0.135" rpy="0 0 0"/>
+       <geometry>
+         <cylinder radius="0.1" length="0.270"/>
+       </geometry>
+       <material name="blue">
+         <color rgba="0.2 0.2 0.8 1.0"/>
+       </material>
+     </visual>
+     <collision>
+       <origin xyz="0 0 0.135" rpy="0 0 0"/>
+       <geometry>
+         <cylinder radius="0.1" length="0.27"/>
+       </geometry>
+     </collision>
+   </link>
+   <joint name="pen_fixed_joint" type="fixed">
+     <parent link="ur5_tool0"/>
+     <child  link="pen_link"/>
+     <!-- ajustez xyz/rpy pour que le stylo corresponde à la réalité -->
+     <origin xyz="0 0 0" rpy="0 0 0"/>
+   </joint>
   </xacro:macro>
 </robot>

Commit message: pb

File: ur5_description_custom/urdf/robot_cell.xacro (robot description, xacro)
@@ -19,5 +19,5 @@
     <link name="table">
       <visual>
-      <origin xyz="0 0 0" rpy="0 0 0"/>
+      <origin xyz="0 0 0.5" rpy="0 0 0"/>
       <geometry>
         <box size="0.8 0.8 1.0"/>
@@ -28,5 +28,5 @@
     </visual>
     <collision>
-      <origin xyz="0 0 0" rpy="0 0 0"/>
+      <origin xyz="0 0 0.5" rpy="0 0 0"/>
       <geometry>
         <box size="0.8 0.8 1.0"/>

Commit message: moins

File: ur5_description_custom/urdf/robot_cell.xacro (robot description, xacro)
@@ -19,5 +19,5 @@
     <link name="table">
       <visual>
-      <origin xyz="0 0 0.5" rpy="0 0 0"/>
+      <origin xyz="0 0 -0.5" rpy="0 0 0"/>
       <geometry>
         <box size="0.8 0.8 1.0"/>

Commit message: flotte

File: ur5_description_custom/urdf/robot_cell.xacro (robot description, xacro)
@@ -38,5 +38,5 @@
       <parent link="table"/>
       <child link="robot_mount"/>
-      <origin xyz="0 0 1.0" rpy="0 0 0" />
+      <origin xyz="0 0 0.5" rpy="0 0 0" />
     </joint>
     <!--This will create the specific robot-->

Commit message: la descente

File: ur5_description_custom/urdf/robot_cell.xacro (robot description, xacro)
@@ -28,5 +28,5 @@
     </visual>
     <collision>
-      <origin xyz="0 0 0.5" rpy="0 0 0"/>
+      <origin xyz="0 0 0" rpy="0 0 0"/>
       <geometry>
         <box size="0.8 0.8 1.0"/>

Commit message: df

File: ur5_description_custom/urdf/robot_cell.xacro (robot description, xacro)
@@ -28,5 +28,5 @@
     </visual>
     <collision>
-      <origin xyz="0 0 0" rpy="0 0 0"/>
+      <origin xyz="0 0 -0.5" rpy="0 0 0"/>
       <geometry>
         <box size="0.8 0.8 1.0"/>
@@ -38,5 +38,5 @@
       <parent link="table"/>
       <child link="robot_mount"/>
-      <origin xyz="0 0 0.5" rpy="0 0 0" />
+      <origin xyz="0 0 0" rpy="0 0 0" />
     </joint>
     <!--This will create the specific robot-->

Commit message: r

File: ur5_description_custom/urdf/robot_cell.xacro (robot description, xacro)
@@ -56,5 +56,5 @@
        <origin xyz="0 0 0.135" rpy="0 0 0"/>
        <geometry>
-         <cylinder radius="0.1" length="0.270"/>
+         <cylinder radius="0.05" length="0.270"/>
        </geometry>
        <material name="blue">
@@ -65,5 +65,5 @@
        <origin xyz="0 0 0.135" rpy="0 0 0"/>
        <geometry>
-         <cylinder radius="0.1" length="0.27"/>
+         <cylinder radius="0.05" length="0.27"/>
        </geometry>
      </collision>
